Commit message: docs:day5 실습 코드 추가

File: mastering_ros_robot_description_pkg/urdf/seven_dof_arm_with_rgbd.xacro (robot description, xacro)
@@ -232,5 +232,5 @@
   </link>
   <gazebo reference="elbow_pitch_link">
-    <material>Gazebo/Red</material>
+    <material>Gazebo/blue</material>
   </gazebo>
   <joint name="wrist_roll_joint" type="revolute">
@@ -318,5 +318,5 @@
   </link>
   <gazebo reference="gripper_roll_link">
-    <material>Gazebo/Red</material>
+    <material>Gazebo/red</material>
   </gazebo>
   <joint name="finger_joint1" type="prismatic">
